Commit message: .

File: src/arm/src/armbot.urdf (robot description, URDF)
Before this commit: robot ArmBot, 6 links, 5 joints
Links:
- added link effector; visual sphere radius=.03
- link elbowLink: geometry visual cylinder length=.05 radius=0.05
- link shoulderALink: geometry visual cylinder length=.05 radius=0.05
- link shoulderBLink: geometry visual cylinder length=.05 radius=0.05
- link wristALink: geometry visual cylinder length=.05 radius=0.05
- link wristBLink: geometry visual cylinder length=0.2 radius=0.01
Joints:
- added joint wristBJoint: type revolute, parent wristBLink, child effector, origin xyz=0 0.2 0 rpy=0 0 0, axis 0 1 0, limit lower=-6.28 upper=6.28 effort=10 velocity=4
- joint elbowJoint: axis 0 0 1 -> 1 0 0; limit lower=-1.308 upper=1.308 effort=10 velocity=4 -> lower=-2 upper=2 effort=10 velocity=4; origin xyz=0 0.3048 0 rpy=0 0 0 -> xyz=0 0.30 0 rpy=0 0 0
- joint shoulderAJoint: origin xyz=0 0 0.381 rpy=0 0 0 -> xyz=0 0 0.3 rpy=0 0 0
- joint shoulderBJoint: axis 0 0 1 -> 1 0 0; limit lower=-1.308 upper=1.308 effort=10 velocity=4 -> lower=-3.1416 upper=3.1416 effort=10 velocity=4
- joint wristAJoint: axis 0 0 1 -> 1 0 0; limit lower=-1.308 upper=1.308 effort=10 velocity=4 -> lower=-3.14 upper=3.14 effort=10 velocity=4; origin xyz=0 0.3048 0 rpy=0 0 0 -> xyz=0 0.30 0 rpy=0 0 0
